File: HDK/SCO68R/SCO68R.kicad_pcb (KiCad board)
At the start: 2 copper layers, 314.4 x 104.3 mm, 181 parts, among them J1 USB C, J2 Conn_01x04, SW1 SW_MEC_5E, SW2 SW_MEC_5E, U1 AMS1117-3.3, U2 TPD4E05U06DQAR, U3 STM32F103C8Tx, Y1 16MHz

Commit message: Edited HDK
Parts:
- added C19: 100nF, Capacitor_SMD:C_0402_1005Metric_Pad0.74x0.62mm_HandSolder, B.Cu at (246.8, -71.3)
- added C20: 100nF, Capacitor_SMD:C_0402_1005Metric_Pad0.74x0.62mm_HandSolder, B.Cu at (246.8, -68.2)
- added C21: 100nF, Capacitor_SMD:C_0402_1005Metric_Pad0.74x0.62mm_HandSolder, B.Cu at (246.8, -65.1)
- added C22: 100nF, Capacitor_SMD:C_0402_1005Metric_Pad0.74x0.62mm_HandSolder, B.Cu at (246.8, -61.9)
- added KSWR3: EC11_RotaryEnc, Rotary_Encoder:RotaryEncoder_Alps_EC11E-Switch_Vertical_H20mm, F.Cu at (251.1, -78.7)
- added KSWR4: EC11_RotaryEnc, Rotary_Encoder:RotaryEncoder_Alps_EC11E-Switch_Vertical_H20mm, F.Cu at (251.1, -59.6)
- added Q1: BSS138, Package_TO_SOT_SMD:SOT-23, B.Cu at (241.5, -80.6)
- added R10: 5k1, Resistor_SMD:R_0402_1005Metric_Pad0.72x0.64mm_HandSolder, B.Cu at (245.6, -100.1)
- added R11: 5k1, Resistor_SMD:R_0402_1005Metric_Pad0.72x0.64mm_HandSolder, B.Cu at (245.6, -71.3)
- added R12: 5k1, Resistor_SMD:R_0402_1005Metric_Pad0.72x0.64mm_HandSolder, B.Cu at (245.6, -68.2)
- added R13: 5k1, Resistor_SMD:R_0402_1005Metric_Pad0.72x0.64mm_HandSolder, B.Cu at (245.6, -65.1)
- added R14: 5k1, Resistor_SMD:R_0402_1005Metric_Pad0.72x0.64mm_HandSolder, B.Cu at (245.6, -61.9)
- added R9: 5k1, Resistor_SMD:R_0402_1005Metric_Pad0.72x0.64mm_HandSolder, B.Cu at (245.6, -103.2)
- C11, C12, C13, C14, R1: moved to F.Cu
- C16, C17, C18: moved to B.Cu
- J2: value Conn_01x04 -> Conn_02x04_Row_Letter_First; footprint Connector_PinHeader_2.54mm:PinHeader_1x04_P2.54mm_Vertical -> Connector_PinHeader_2.54mm:PinHeader_2x04_P2.54mm_Vertical; moved to B.Cu
- R5, R6: value 5k1 -> 10k
- moved R7 190.3 mm to (245.6, -109.5), turned to -90 degrees
- moved C15 187.1 mm to (246.8, -109.5), turned to -90 degrees
- moved C14 186.8 mm to (239.7, -114.2), turned to 90 degrees
- moved R8 184.5 mm to (245.6, -106.3), turned to -90 degrees
- moved C12 182.5 mm to (239.7, -92.1), turned to 90 degrees
- moved R5 181.1 mm to (241.5, -77.8)
- moved C13 180.7 mm to (239.7, -103.1), turned to 90 degrees
- moved R6 174.1 mm to (239.0, -80.5), turned to 90 degrees
- moved J2 73.1 mm to (100.6, -39.3), turned to -90 degrees
- moved C11 48.3 mm to (112.8, -40.3), turned to 0 degrees
- moved C10 42.2 mm to (55.8, -32.0), turned to -90 degrees
- moved D58 36.3 mm to (258.8, -47.8), turned to 0 degrees
- moved C1 20.2 mm to (29.6, -43.1), turned to 0 degrees
- moved SW2 19.0 mm to (118.9, -42.2), turned to 180 degrees
- moved D15 17.4 mm to (258.6, -104.8), turned to 0 degrees
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Connections:
- C10 pad 1: GND -> +3.3V
- C10 pad 2: NRST -> GND
- C11 pad 1: +3.3V -> GND
- C11 pad 2: GND -> NRST
- C12 pad 1: GND -> +5V
- C12 pad 2: ROT1_A -> GND
- C13 pad 1: GND -> +5V
- C13 pad 2: ROT2_A -> GND
- C14 pad 1: ROT1_B -> +5V
- C15 pad 1: ROT2_B -> ROT1_A
- C16 pad 1: +5V -> ROT1_B
- C17 pad 1: +5V -> ROT2_A
- C18 pad 1: +5V -> ROT2_B
- J2 pad 1: GND -> +3.3V
- J2 pad 2: SWCLK -> +3.3V
- J2 pad 4: +3.3V -> BOOT0
- R5 pad 1: ROT1_A -> +3.3V
- R5 pad 2: +3.3V -> NEOPIXEL_DRIVE_L
- R6 pad 1: ROT2_A -> +5V
- R6 pad 2: +3.3V -> NEOPIXEL_DRIVE_H
- R7 pad 1: ROT1_B -> ROT1_A
- R8 pad 1: ROT2_B -> ROT1_B
- U3 pad 10: COL 0 -> COL 14
- U3 pad 11: COL 1 -> ROW 4
- U3 pad 12: COL 2 -> unconnected-(U3-Pad12)
- U3 pad 13: ROW 4 -> unconnected-(U3-Pad13)
- U3 pad 14: unconnected-(U3-Pad14) -> COL 7
- U3 pad 15: unconnected-(U3-Pad15) -> COL 8
- U3 pad 16: unconnected-(U3-Pad16) -> ROW 0
- U3 pad 17: unconnected-(U3-Pad17) -> ROW 1
- U3 pad 18: unconnected-(U3-Pad18) -> ROW 2
- U3 pad 19: unconnected-(U3-Pad19) -> ROW 3
- U3 pad 2: unconnected-(U3-Pad2) -> COL 11
- U3 pad 20: unconnected-(U3-Pad20) -> COL 4
- U3 pad 21: unconnected-(U3-Pad21) -> COL 5
- U3 pad 22: unconnected-(U3-Pad22) -> COL 6
- U3 pad 25: unconnected-(U3-Pad25) -> COL 3
- U3 pad 26: unconnected-(U3-Pad26) -> COL 2
- U3 pad 27: unconnected-(U3-Pad27) -> COL 1
- U3 pad 28: ROW 2 -> COL 0
- U3 pad 29: ROW 1 -> ROT4_A
- U3 pad 3: unconnected-(U3-Pad3) -> COL 12
- U3 pad 30: ROW 0 -> ROT4_B
- U3 pad 31: ROW 3 -> NEOPIXEL_DRIVE_L
- U3 pad 38: ROT1_A -> ROT3_A
- U3 pad 39: ROT1_B -> ROT3_B
- U3 pad 4: unconnected-(U3-Pad4) -> COL 13
- U3 pad 40: ROT2_A -> ROT1_A
- U3 pad 41: ROT2_B -> ROT1_B
- U3 pad 42: NEOPIXEL_DRIVE_H -> ROT2_A
- U3 pad 43: unconnected-(U3-Pad43) -> ROT2_B
- U3 pad 45: unconnected-(U3-Pad45) -> COL 9
- U3 pad 46: unconnected-(U3-Pad46) -> COL 10
Routing:
- net +3.3V: track 252.9 -> 497.1 mm, vias 13 -> 15
- net ROT3_A: track 0.00 -> 211.6 mm, vias 0 -> 2
- net ROT4_A: track 0.00 -> 210.6 mm, vias 0 -> 2
- net ROT4_B: track 0.00 -> 210.2 mm, vias 0 -> 2
- net NEOPIXEL_DRIVE_L: track 0.00 -> 206.2 mm, vias 0 -> 2
- net ROT3_B: track 0.00 -> 206.2 mm, vias 0 -> 2
- net NEOPIXEL_DRIVE_H: track 206.0 -> 11.5 mm
- net COL 14: track 155.6 -> 324.8 mm, vias 0 -> 2
- net COL 13: track 126.1 -> 292.2 mm, vias 1 -> 2
- net COL 12: track 106.5 -> 267.9 mm, vias 0 -> 2
- net COL 11: track 95.0 -> 244.8 mm, vias 0 -> 2
- net COL 10: track 90.6 -> 223.0 mm, vias 0 -> 2
- net COL 9: track 90.6 -> 206.0 mm, vias 0 -> 2
- net COL 8: track 66.0 -> 159.6 mm, vias 0 -> 2
- net COL 7: track 66.0 -> 139.6 mm, vias 0 -> 2
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