File: HDK/SCO68R/V1/SCO68R_V1.kicad_sch (KiCad schematic)
At the start: 190 parts, among them J1 USB C, J2 Conn_02x04_Row_Letter_First, Q1 BSS138, SW1 SW_MEC_5E, SW2 SW_MEC_5E, U1 AMS1117-3.3, U2 TPD4E05U06DQAR, U3 STM32F103C8Tx, Y1 16MHz

Commit message: Edited HDK
Parts:
- removed C16, C17, C18, C19, C20, C21, C22: 100nF, Capacitor_SMD:C_0402_1005Metric_Pad0.74x0.62mm_HandSolder, symbol Device:C
- removed J2: Conn_02x04_Row_Letter_First, Connector_PinHeader_2.54mm:PinHeader_2x04_P2.54mm_Vertical, symbol Connector_Generic:Conn_02x04_Odd_Even
- removed KSWR3, KSWR4: EC11_RotaryEnc, Rotary_Encoder:RotaryEncoder_Alps_EC11E-Switch_Vertical_H20mm, symbol 0SCO_LIB:EC11_RotaryEnc
- removed Q1: BSS138, Package_TO_SOT_SMD:SOT-23, symbol Transistor_FET:BSS138
- removed R10, R11, R12, R13, R14, R9: 5k1, Resistor_SMD:R_0402_1005Metric_Pad0.72x0.64mm_HandSolder, symbol Device:R
- added C12, C13, C14: 100nF, Capacitor_SMD:C_0402_1005Metric_Pad0.74x0.62mm_HandSolder, symbol Device:C
- added J2: Conn_01x04, Connector_PinHeader_2.54mm:PinHeader_1x04_P2.54mm_Vertical, symbol Connector_Generic:Conn_01x04
- R5, R6: value 10k -> 5k1
- renumbered C11 to C10, C10 to C11, C12 to C16, C13 to C17, C14 to C18
Connections:
- net ROT3_A is gone; now on net ROT1_A: U3.38 (PA15)
- net ROT3_B is gone; now on net ROT1_B: U3.39 (PB3)
- net ROT4_A is gone; now on net ROW 1: U3.29 (PA8)
- net ROT4_B is gone; now on net ROW 0: U3.30 (PA9)
- net +3.3V: now also R5.2, R6.2, J2.4 (Pin_4); no longer R5.1
- net +5V: no longer R6.1
- net COL 0: now also U3.10 (PA0); no longer U3.28 (PB15)
- net COL 1: now also U3.11 (PA1); no longer U3.27 (PB14)
- net COL 10: no longer U3.46 (PB9)
- net COL 11: no longer U3.2 (PC13)
- net COL 12: no longer U3.3 (PC14)
- net COL 13: no longer U3.4 (PC15)
- net COL 14: no longer U3.10 (PA0)
- net COL 2: now also U3.12 (PA2); no longer U3.26 (PB13)
- net COL 3: no longer U3.25 (PB12)
- net COL 4: no longer U3.20 (PB2)
- net COL 5: no longer U3.21 (PB10)
- net COL 6: no longer U3.22 (PB11)
- net COL 7: no longer U3.14 (PA4)
- net COL 8: no longer U3.15 (PA5)
- net COL 9: no longer U3.45 (PB8)
- net GND: now also C12.1, C13.1, C14.2, J2.1 (Pin_1)
- net NEOPIXEL_DRIVE_H: now also U3.42 (PB6); no longer R6.2
- net ROT1_A: now also R5.1, C12.2; no longer C15.1, R7.1, U3.40 (PB4)
- net ROT1_B: now also R7.1, C14.1; no longer R8.1, U3.41 (PB5)
- net ROT2_A: now also R6.1, U3.40 (PB4), C13.2; no longer U3.42 (PB6)
- net ROT2_B: now also C15.1, R8.1, U3.41 (PB5); no longer U3.43 (PB7)
- net ROW 0: no longer U3.16 (PA6)
- net ROW 1: no longer U3.17 (PA7)
- net ROW 2: now also U3.28 (PB15); no longer U3.18 (PB0)
- net ROW 3: now also U3.31 (PA10); no longer U3.19 (PB1)
- net ROW 4: now also U3.13 (PA3); no longer U3.11 (PA1)
- net SWCLK: now also J2.2 (Pin_2)
- net SWDIO: now also J2.3 (Pin_3)
- removed net NEOPIXEL_DRIVE_L: R5.2, U3.31 (PA10)
Other:
- note removed: "Decoupling Caps for Neopixels"
- note removed: "Level Shifter for Neopixels"
- note removed: "Rotary Encoder Debounce"
- moved on the sheet: C16, C17, C18, C3, C4, D69, D70, D71, Y1
